File: tools/autoroute/base-routed.kicad_pcb (KiCad board)
At the start: 4 copper layers, 66 x 100 mm, 78 parts, among them J1 USB_C_Receptacle_USB2.0_14P, J10 SM09B-SRSS-TB, J11 SM06B-SRSS-TB, J4 SM06B-SRSS-TB, J5 SM06B-SRSS-TB, J6 SM06B-SRSS-TB, J7 SM06B-SRSS-TB, J8 S6B-PH-K, J9 S6B-PH-K, Q1 AO4407A, SW1 SW_Push, SW2 SW_Push, SW3 JS102011SAQN, U1 ESP32-S3-WROOM-1-N16, U2 USBLC6-2SC6, U3 AP63203WU, U4 DRV8231ADSG, U5 DRV8231ADSG

Commit message: layout: rework the motor region for review findings 1-3
REVIEW.md found undersized motor-output copper, a poor heat path out of the
driver exposed pads, and bypass capacitors too far from VM to close a local
loop. tools/autoroute/rework.py fixes all three in one reproducible pass over
base-routed.kicad_pcb, a snapshot of the original routing.

1. Motor copper. MOT_B_1 carried 38.8 of its 42 mm at 0.15 mm, MOT_B_2 41.3 of
   48 mm. All four nets are now 0.8 mm trunks, with 0.2-0.4 mm only inside the
   drivers' own pin field. The motor-B pair goes 0.267 -> 0.062 ohm, so at the
   DRV8231A's 1.47 A limit 0.393 V / 0.578 W become 0.090 V / 0.133 W. A Motor
   netclass and the new Pixy-M2.kicad_dru enforce >= 0.6 mm outside two named
   "Motor pin escape" rule areas, so the next long neck fails DRC instead of
   passing it. The rule uses enclosedByArea, not intersectsArea: with
   intersects, a trunk that merely starts in the area is exempt along its whole
   length, which was observed and fixed.

2. Exposed pads. U4's had no via in it at all and U5's had one. Each now has
   two in-pad thermal vias at 0.45/0.25 - the board's own minimum via, and all
   that the 0.45 mm hole-to-hole rule allows in a 0.9 x 1.6 mm pad - plus
   0.8 mm copper out of the pad, four GND vias within 3 mm, and a new F.Cu
   pour putting 165 mm^2 of ground copper around both drivers.

3. Bypass loops. C18 and C20 sat 4.95 mm and 3.61 mm from their VM pin and
   reached it only through the In2 plane, 1.065 mm of core away from the In1
   return. Both are now 1.33 mm away, across pins 5 and 7, with the loop closed
   entirely in top copper. C21 moved to clear the escape corridor that created.

DRC is unchanged from before the rework: 0 unconnected items, 0 schematic
parity issues, and only the four pre-existing J1 hole_clearance errors and the
pre-existing U1 lib_footprint_mismatch warning.

Not addressed: finding 4 - U5 is still ~40 mm from J9 and the motor-B outputs
are still not routed as a pai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
Parts:
- moved C21 7.80 mm to (113.0, 114.0)
- moved C18 6.17 mm to (106.0, 111.0)
- moved C20 3.34 mm to (120.0, 111.0)
Routing:
- net GND: track 78.4 -> 72.8 mm, vias 84 -> 77
- net /MOT_A_2: track 19.0 -> 16.2 mm
- net /MOT_A_1: track 16.7 -> 15.0 mm
- net /MOT_B_1: track 43.5 -> 41.9 mm, vias 1 -> 0
- net /VBAT: track 68.2 -> 69.1 mm, vias 24 -> 27
- net /MOT_B_2: track 48.6 -> 48.1 mm, vias 2 -> 0
- removed copper zone on F.Cu, net GND
