File: Pixy-M2.kicad_sch (KiCad schematic)
At the start: 58 parts, among them J1 USB_C_Receptacle_USB2.0_14P, J2 Conn_01x22_Pin, J3 Conn_01x22_Pin, J4 SM06B-SRSS-TB, J5 SM06B-SRSS-TB, J6 SM06B-SRSS-TB, J7 SM06B-SRSS-TB, Q1 AO4407A, SW1 SW_Push, SW2 SW_Push, SW3 JS102011SAQN, U1 ESP32-S3-WROOM-1-N16, U2 USBLC6-2SC6, U3 AP63203WU

Commit message: Remove series resistors from USB D+/D- (issue 10)
R3 and R4 (22 ohm) sat between U2 and the module's USB pins and did
nothing: the ESP32-S3's USB PHY is internally impedance-matched and
Espressif's reference designs connect straight through. Deleted both
symbols and joined the wires so U2 drives U1 directly.

Deleted rather than set to 0 ohm. Both were sanctioned by the original
note; removal won because two 0805 jumper pads are a discontinuity in the
90 ohm differential pair the layout rules call for, sitting exactly where
routing is tightest next to the USB-C connector. At Full Speed (12 Mbps)
that discontinuity would have been harmless in practice -- this is about
keeping the pair clean and the BOM short, not fixing a real defect.

Verified:
- Netlist diff shows exactly four changes: /USB_D+ absorbed U2.4,
  /USB_D- absorbed U2.6, and the auto-named Net-(R3-Pad2) and
  Net-(R4-Pad1) disappeared. Net count 64 -> 62 as expected.
- ERC unchanged at 0 errors, 0 warnings.
- Sheet rendered and inspected: both runs go straight from U2 to their
  labels with no junction picked up. The wire-through-a-junction hazard
  that has bitten this board twice did not recur.

Co-Authored-By: Claude Opus 5 <noreply@anthropic.com>
Parts:
- removed R3, R4: 22Ohm, Resistor_SMD:R_0805_2012Metric, symbol Device:R_US
Connections:
- net USB_D+: now also U2.4 (I/O2)
- net USB_D-: now also U2.6 (I/O1)
Changed lines of the file:
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@@
 	(wire
 		(pts
-			(xy 99.06 168.91) (xy 99.06 171.45)
-		)
-		(stroke
-			(width 0)
-			(type default)
-		)
-	)
-	(wire
-		(pts
 			(xy 87.63 137.16) (xy 93.98 137.16)
 		)
@@
 	(wire
 		(pts
-			(xy 111.76 168.91) (xy 111.76 171.45)
-		)
-		(stroke
-			(width 0)
-			(type default)
-		)
-	)
-	(wire
-		(pts
 			(xy 60.96 144.78) (xy 63.5 144.78)
 		)
@@
 	(wire
 		(pts
-			(xy 111.76 161.29) (xy 111.76 152.4)
+			(xy 111.76 171.45) (xy 111.76 152.4)
 		)
 		(stroke
@@
 	(wire
 		(pts
-			(xy 99.06 154.94) (xy 99.06 161.29)
+			(xy 99.06 154.94) (xy 99.06 171.45)
 		)
 		(stroke
@@
 	)
 	(symbol
-		(lib_id "Device:R_US")
-		(at 99.06 165.1 0)
-		(unit 1)
-		(body_style 1)
-		(exclude_from_sim no)
-		(in_bom yes)
-		(on_board yes)
-		(in_pos_files yes)
-		(dnp no)
-		(fields_autoplaced yes)
-		(property "Reference" "R4"
-			(at 101.6 163.8299 0)
-			(show_name no)
-			(do_not_autoplace no)
-			(effects
-				(font
-					(size 1.27 1.27)
-				)
-				(justify left)
-			)
-		)
-		(property "Value" "22Ohm"
-			(at 101.6 166.3699 0)
-			(show_name no)
-			(do_not_autoplace no)
-			(effects
-				(font
-					(size 1.27 1.27)
-				)
-				(justify left)
-			)
-		)
-		(property "Footprint" "Resistor_SMD:R_0805_2012Metric"
-			(at 100.076 165.354 90)
-			(hide yes)
-			(show_name no)
-			(do_not_autoplace no)
-			(effects
-				(font
-					(size 1.27 1.27)
-				)
-			)
-		)
-		(property "Datasheet" ""
-			(at 99.06 165.1 0)
-			(hide yes)
-			(show_name no)
-			(do_not_autoplace no)
-			(effects
-				(font
-					(size 1.27 1.27)
-				)
-			)
-		)
-		(property "Description" "Resistor, US symbol"
-			(at 99.06 165.1 0)
-			(hide yes)
-			(show_name no)
-			(do_not_autoplace no)
-			(effects
-				(font
-					(size 1.27 1.27)
-				)
-			)
-		)
-		(pin "1"
-		)
-		(pin "2"
-		)
-		(instances
-			(project "Pixy-M2"
-				(path "/fefb2c5c-cd05-4562-bf27-32a51f81fd04"
-					(reference "R4")
-					(unit 1)
-				)
-			)
-		)
-	)
-	(symbol
 		(lib_id "power:GND")
 		(at 81.28 124.46 0)
@@
 					(unit 1)
 				)
-			)
-		)
-	)
-	(symbol
-		(lib_id "Device:R_US")
-		(at 111.76 165.1 180)
-		(unit 1)
-		(body_style 1)
-		(exclude_from_sim no)
-		(in_bom yes)
-		(on_board yes)
-		(in_pos_files yes)
-		(dnp no)
-		(fields_autoplaced yes)
-		(property "Reference" "R3"
-			(at 114.3 163.8299 0)
-			(show_name no)
-			(do_not_autoplace no)
-			(effects
-				(font
-					(size 1.27 1.27)
-				)
-				(justify right)
-			)
-		)
-		(property "Value" "22Ohm"
-			(at 114.3 166.3699 0)
-			(show_name no)
-			(do_not_autoplace no)
-			(effects
-				(font
-					(size 1.27 1.27)
-				)
-				(justify right)
-			)
-		)
-		(property "Footprint" "Resistor_SMD:R_0805_2012Metric"
-			(at 110.744 164.846 90)
-			(hide yes)
-			(show_name no)
-			(do_not_autoplace no)
-			(effects
-				(font
-					(size 1.27 1.27)
-				)
-			)
-		)
-		(property "Datasheet" ""
-			(at 111.76 165.1 0)
-			(hide yes)
-			(show_name no)
-			(do_not_autoplace no)
-			(effects
-				(font
-					(size 1.27 1.27)
-				)
-			)
-		)
-		(property "Description" "Resistor, US symbol"
-			(at 111.76 165.1 0)
-			(hide yes)
-			(show_name no)
-			(do_not_autoplace no)
-			(effects
-				(font
-					(size 1.27 1.27)
-				)
-			)
-		)
-		(pin "1"
-		)
-		(pin "2"
-		)
-		(instances
-			(project "Pixy-M2"
-				(path "/fefb2c5c-cd05-4562-bf27-32a51f81fd04"
-					(reference "R3")
-					(unit 1)
-				)

Commit message: Specify real parts for OR-ing diodes D1/D2 (issue 9)
Both were Value "D_Schottky" with an empty Datasheet field. Both are now
onsemi MBRA340T3G -- same part in both positions, since the requirements
and footprint are identical and it saves a BOM line and a reel. Value,
MPN, Datasheet and Description populated together, following D3/BAT54W.

Verified against the onsemi datasheet (MBRA340T3/D Rev. 12) rather than
from memory: SMA / CASE 403D (DO-214AC), VRRM 40V, IO 3.0A at TL = 100C,
IFSM 100A, VF 0.450V max at 3.0A/25C, IR 0.3mA at 40V/25C, RthJA 81 C/W.

Corrects this issue's premise, which was wrong. It claimed D2 carries the
entire system current (~1A, ~400mW) and on that basis floated replacing it
with a P-FET ideal-diode controller. The netlist says VSYS has exactly four
members -- C12.1, D1.1, D2.1, U3.3(IN) -- so D2 feeds the buck input only;
motor current reaches J2.19-22 in parallel with it. Worst case is ~0.43A
and ~140mW, so the ideal-diode option is unnecessary and is recorded as
such so it is not re-proposed.

Also records the package trap that caught this change: "SS34" is the
obvious commodity answer but Vishay's SS34 is SMC (DO-214AB), not the SMA
this footprint needs. Other makers sell an SMA "SS34", so the part number
alone does not pin down the package.

Verified:
- Netlist diff: no net changed, count steady at 62. Field-only edit, as
  intended.
- ERC unchanged at 0 errors, 0 warnings.
- Sheet rendered and inspected: both Value strings render clear of the
  diode bodies and neighbouring text.

Co-Authored-By: Claude Opus 5 <noreply@anthropic.com>
Parts:
- D1, D2: value D_Schottky -> MBRA340T3G; MPN (none) -> MBRA340T3G
Changed lines of the file:
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@@
 			)
 		)
-		(property "Value" "D_Schottky"
+		(property "Value" "MBRA340T3G"
 			(at 158.75 101.9174 90)
 			(show_name no)
@@
 			)
 		)
-		(property "Datasheet" ""
+		(property "Datasheet" "https://www.onsemi.com/pdf/datasheet/mbra340t3-d.pdf"
 			(at 156.21 100.33 0)
 			(hide yes)
@@
 			)
 		)
-		(property "Description" "Schottky diode"
+		(property "Description" "40V 3A Schottky barrier rectifier, DO-214AC/SMA. VF 0.450V max at 3.0A/25C; IFSM 100A; IR 0.3mA at 40V/25C. K=1, A=2."
 			(at 156.21 100.33 0)
 			(hide yes)
 			(show_name no)
 			(do_not_autoplace no)
+			(effects
+				(font
+					(size 1.27 1.27)
+				)
+			)
+		)
+		(property "MPN" "MBRA340T3G"
+			(at 156.21 100.33 0)
+			(hide yes)
 			(effects
 				(font
@@
 			)
 		)
-		(property "Value" "D_Schottky"
+		(property "Value" "MBRA340T3G"
 			(at 98.1075 133.35 0)
 			(show_name no)
@@
 			)
 		)
-		(property "Datasheet" ""
+		(property "Datasheet" "https://www.onsemi.com/pdf/datasheet/mbra340t3-d.pdf"
 			(at 97.79 137.16 0)
 			(hide yes)
@@
 			)
 		)
-		(property "Description" "Schottky diode"
+		(property "Description" "40V 3A Schottky barrier rectifier, DO-214AC/SMA. VF 0.450V max at 3.0A/25C; IFSM 100A; IR 0.3mA at 40V/25C. K=1, A=2."
 			(at 97.79 137.16 0)
 			(hide yes)
@@
 			(effects
 				(font
+					(size 1.27 1.27)
+				)
+			)
+		)
+		(property "MPN" "MBRA340T3G"
+			(at 97.79 137.16 0)
+			(hide yes)
+			(effects
+				(font
